File: ReFloMatic.kicad_pcb (KiCad board)
At the start: 2 copper layers, 54.4 x 85.3 mm, 151 parts, among them CON2 MicroSD_Card, P1 PROG, P2 THERMOCOUPLE, P3 DOOR_SERVO, P4 OVEN, P5 USB_B, P6 PWR_CONN, Q1 MMUN2211, Q2 MMUN2111, Q3 MMUN2111, Q4 MMUN2211, U1 STM32F030C, U2 MAX31855KASA

Commit message: Changed internal cutout to board edge layer.  Regenerated gerbers.  Ordered PCB.
Other:
- outline, holes or cut-outs redrawn
- board text added: "CUT OUT"
Changed lines of the file:
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@@
 (kicad_pcb (version 4) (host pcbnew 4.0.1-stable)
   (general
-    (links 0)
+    (links 304)
     (no_connects 0)
     (area 122.428514 61.7246 183.946286 149.7836)
     (thickness 1.6)
-    (drawings 28)
+    (drawings 33)
     (tracks 666)
     (zones 0)
@@
     (trace_min 0.1524)
     (segment_width 0.2)
-    (edge_width 0.15)
+    (edge_width 0.001)
     (via_size 0.6858)
     (via_drill 0.3302)
@@
     (visible_elements 7FFFFF7F)
     (pcbplotparams
-      (layerselection 0x010f0_80000001)
+      (layerselection 0x218f0_80000001)
       (usegerberextensions true)
       (excludeedgelayer true)
@@
     (add_net "Net-(U1-Pad7)")
   )
-  (module TFT:ER-TFT028-4 locked (layer F.Cu)
+  (module TFT:ER-TFT028-4 (layer F.Cu)
     (at 153.25 115.7)
     (fp_text reference DS1 (at -0.05 -2.8) (layer F.SilkS)
@@
     (pad 0 smd rect (at 13.79 1.45) (size 2 4) (layers F.Cu F.Paste F.Mask)
       (net 4 GND))
-    (pad "" np_thru_hole oval (at 0 11.85) (size 30 6) (drill oval 30 6) (layers *.Cu)
-      (zone_connect 0))
     (pad "" np_thru_hole circle (at 23.52 -44) (size 1 1) (drill 1) (layers *.Cu))
     (pad "" np_thru_hole circle (at -23.52 -44) (size 1 1) (drill 1) (layers *.Cu))
@@
       (net 4 GND) (zone_connect 2))
   )
-  (module TFT:ER-TFT028-4 locked (layer F.Cu)
+  (module TFT:ER-TFT028-4 (layer F.Cu)
     (at 153.25 115.7)
     (fp_text reference DS1 (at -0.05 -2.8) (layer F.SilkS)
@@
     (pad 0 smd rect (at 13.79 1.45) (size 2 4) (layers F.Cu F.Paste F.Mask)
       (net 4 GND))
-    (pad "" np_thru_hole oval (at 0 11.85) (size 30 6) (drill oval 30 6) (layers *.Cu)
-      (zone_connect 0))
     (pad "" np_thru_hole circle (at 23.52 -44) (size 1 1) (drill 1) (layers *.Cu))
     (pad "" np_thru_hole circle (at -23.52 -44) (size 1 1) (drill 1) (layers *.Cu))
@@
       (xy 7.093862 -0.807174) (xy 7.173264 -0.780087)) (layer F.SilkS) (width 0.01))
   )
+  (gr_text "CUT OUT" (at 153 127.8) (layer Eco2.User)
+    (effects (font (size 3 3) (thickness 0.3)))
+  )
+  (gr_line (start 138.2 130.6) (end 138.2 124.6) (layer Edge.Cuts) (width 0.001))
+  (gr_line (start 168.2 130.6) (end 138.2 130.6) (layer Edge.Cuts) (width 0.001))
+  (gr_line (start 168.2 124.6) (end 168.2 130.6) (layer Edge.Cuts) (width 0.001))
+  (gr_line (start 138.2 124.6) (end 168.2 124.6) (layer Edge.Cuts) (width 0.001))
   (gr_text TX (at 157.3784 89.916 90) (layer F.SilkS)
     (effects (font (size 0.8 0.8) (thickness 0.16)) (justify right))
